File: EEG/PCB_Circuits/Hardware_Comp_V1.4.sch (EAGLE design)
At the start: 17 parts, among them IC1 LMV324M, U1 AD8422ARMZRM_8-L

Commit message: Version_4
Parts:
- removed IC1: LMV324M, linear:LMV324M
- added C10: 2.2u, adafruit:C-USC0603
- added C11: 1u, adafruit:C-USC0603
- added C12, C13: 0.1u, adafruit:C-USC0603
- added C16: 10u, adafruit:C-USC0603
- added C9: 0.12u, adafruit:C-USC0603
- added R10: 400K, adafruit:R-US_R0603
- added R11, R9: 3.4K, adafruit:R-US_R0603
- added R12: 60.4K, adafruit:R-US_R0603
- added R4: 10K, adafruit:R-US_R0603
- added R5, R6: 20K, adafruit:R-US_R0603
- added R7, R8: 5K, adafruit:R-US_R0603
- added U2, U3, U4: LMV324, SparkFun-IC-Amplifiers:LMV324
- C6: value 10u -> 0.1u
- R2: value 37.4K -> 75K
- R3: value 50 -> 37.4K
Connections:
- removed net V+: 9V-.1, C3.2, C4.2, C7.1, IC1P.V+, U1.+VS
- removed net V-: C1.2, C2.2, IC1P.V-, JP3.1, U1.-VS
- new net N$10: R5.1, R6.2, U3G2.-IN
- new net N$11: C9.2, R4.1, U3G2.+IN
- new net N$13: R10.1
- new net N$14: C9.1, R8.1, U3G4.+IN
- new net N$15: C10.1, R7.1, R8.2
- new net N$17: C12.2, R12.1, U3G3.+IN
- new net N$18: C11.2, R4.2, R5.2, U3G3.-IN, U3G3.OUT
- new net N$19: C11.1, R11.1, R12.2
- new net N$7: R6.1, U3G1.+IN, U3G2.OUT
- new net N$8: C10.2, U3G4.-IN, U3G4.OUT
- new net V+2: C1.2, C2.2, C7.1, JP3.1, U1.-VS, U2G5.P$V-, U4G5.P$V-
- new net V+3: C8.1
- new net V+4: C13.1
- net GND: now also C12.1, C13.2, C6.2, R2.2, R7.2, R9.2; no longer R3.1
- net N$1: now also C16.1, C5.1, R3.2
- net N$2: now also R11.2, R3.1, U2G1.-IN, U2G1.OUT; no longer C5.1, C6.1, R2.2
- net N$3: now also C16.2, R2.1, U2G1.+IN; no longer C6.2, IC1A.+IN, R3.2
- net N$4: now also R10.2, R9.1, U3G1.-IN; no longer IC1A.-IN, IC1A.OUT, R2.1
- net V+1: now also 9V-.1, C3.2, C4.2, C6.1, U1.+VS, U2G5.P$V+, U4G5.P$V+; no longer C8.1
Other:
- moved on the sheet: C5, C6, C7, C8, R2, R3

Commit message: Created Board file for version 4
Connections:
- removed net V+1: 9V-.1, C3.2, C4.2, C6.1, U1.+VS, U2G5.P$V+, U4G5.P$V+
- removed net V+2: C1.2, C2.2, C7.1, JP3.1, U1.-VS, U2G5.P$V-, U4G5.P$V-
- net V+3: now also 9V-.1, C3.2, C4.2, C6.1, U1.+VS, U2G5.P$V+, U4G5.P$V+
- net V+4: now also C1.2, C2.2, C7.1, JP3.1, U1.-VS, U2G5.P$V-, U4G5.P$V-
Changed lines of the file:
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@@
 <pinref part="U1" gate="A" pin="VOUT"/>
 <wire x1="-12.7" y1="71.12" x2="-12.7" y2="40.64" width="0.1524" layer="91"/>
-<wire x1="20.32" y1="40.64" x2="33.02" y2="40.64" width="0.1524" layer="91"/>
 <pinref part="C5" gate="G$1" pin="2"/>
 <pinref part="C5" gate="G$1" pin="1"/>
@@
 <wire x1="-12.7" y1="40.64" x2="12.7" y2="40.64" width="0.1524" layer="91"/>
 <junction x="12.7" y="40.64"/>
+<wire x1="20.32" y1="40.64" x2="33.02" y2="40.64" width="0.1524" layer="91"/>
+<junction x="20.32" y="40.64"/>
 </segment>
 </net>
@@
 </segment>
 </net>
-<net name="V+1" class="0">
-<segment>
+<net name="N$2" class="0">
+<segment>
+<wire x1="60.96" y1="45.72" x2="50.8" y2="45.72" width="0.1524" layer="91"/>
+<wire x1="50.8" y1="45.72" x2="50.8" y2="63.5" width="0.1524" layer="91"/>
+<wire x1="76.2" y1="43.18" x2="81.28" y2="43.18" width="0.1524" layer="91"/>
+<wire x1="81.28" y1="43.18" x2="91.44" y2="43.18" width="0.1524" layer="91"/>
+<wire x1="91.44" y1="43.18" x2="91.44" y2="68.58" width="0.1524" layer="91"/>
+<wire x1="50.8" y1="63.5" x2="81.28" y2="63.5" width="0.1524" layer="91"/>
+<wire x1="81.28" y1="63.5" x2="81.28" y2="43.18" width="0.1524" layer="91"/>
+<junction x="81.28" y="43.18"/>
+<wire x1="91.44" y1="68.58" x2="71.12" y2="68.58" width="0.1524" layer="91"/>
+<wire x1="71.12" y1="68.58" x2="68.58" y2="68.58" width="0.1524" layer="91"/>
+<wire x1="91.44" y1="43.18" x2="99.06" y2="43.18" width="0.1524" layer="91"/>
+<junction x="91.44" y="43.18"/>
+<pinref part="U2" gate="G1" pin="-IN"/>
+<pinref part="U2" gate="G1" pin="OUT"/>
+<pinref part="R3" gate="G$1" pin="1"/>
+<junction x="71.12" y="68.58"/>
+<pinref part="R11" gate="G$1" pin="2"/>
+</segment>
+</net>
+<net name="N$3" class="0">
+<segment>
+<wire x1="50.8" y1="40.64" x2="60.96" y2="40.64" width="0.1524" layer="91"/>
+<wire x1="50.8" y1="40.64" x2="50.8" y2="38.1" width="0.1524" layer="91"/>
+<pinref part="U2" gate="G1" pin="+IN"/>
+<pinref part="C16" gate="G$1" pin="2"/>
+<wire x1="50.8" y1="38.1" x2="50.8" y2="33.02" width="0.1524" layer="91"/>
+<wire x1="43.18" y1="40.64" x2="50.8" y2="40.64" width="0.1524" layer="91"/>
+<junction x="50.8" y="40.64"/>
+<pinref part="R2" gate="G$1" pin="1"/>
+<junction x="50.8" y="38.1"/>
+</segment>
+</net>
+<net name="V+3" class="0">
+<segment>
+<wire x1="388.62" y1="106.68" x2="396.24" y2="106.68" width="0.1524" layer="91"/>
+<pinref part="C8" gate="G$1" pin="1"/>
 <wire x1="27.94" y1="106.68" x2="35.56" y2="106.68" width="0.1524" layer="91"/>
 <pinref part="C6" gate="G$1" pin="1"/>
@@
 <wire x1="-76.2" y1="81.28" x2="-76.2" y2="58.42" width="0.1524" layer="91"/>
 <wire x1="-99.06" y1="137.16" x2="27.94" y2="137.16" width="0.1524" layer="91"/>
-<wire x1="27.94" y1="137.16" x2="388.62" y2="137.16" width="0.1524" layer="91"/>
+<wire x1="27.94" y1="137.16" x2="388.62" y2="139.7" width="0.1524" layer="91"/>
 <pinref part="U2" gate="G5" pin="P$V+"/>
 <wire x1="27.94" y1="106.68" x2="27.94" y2="137.16" width="0.1524" layer="91"/>
 <junction x="27.94" y="137.16"/>
 <pinref part="U4" gate="G5" pin="P$V+"/>
-<wire x1="388.62" y1="137.16" x2="388.62" y2="106.68" width="0.1524" layer="91"/>
-</segment>
-</net>
-<net name="V+2" class="0">
-<segment>
+<wire x1="388.62" y1="139.7" x2="388.62" y2="106.68" width="0.1524" layer="91"/>
+<junction x="388.62" y="106.68"/>
+<junction x="27.94" y="106.68"/>
+</segment>
+</net>
+<net name="V+4" class="0">
+<segment>
+<wire x1="388.62" y1="91.44" x2="396.24" y2="91.44" width="0.1524" layer="91"/>
+<pinref part="C13" gate="G$1" pin="1"/>
 <wire x1="27.94" y1="91.44" x2="35.56" y2="91.44" width="0.1524" layer="91"/>
 <pinref part="C7" gate="G$1" pin="1"/>
@@
 <pinref part="U4" gate="G5" pin="P$V-"/>
 <wire x1="388.62" y1="91.44" x2="388.62" y2="-40.64" width="0.1524" layer="91"/>
-</segment>
-</net>
-<net name="N$2" class="0">
-<segment>
-<wire x1="60.96" y1="45.72" x2="50.8" y2="45.72" width="0.1524" layer="91"/>
-<wire x1="50.8" y1="45.72" x2="50.8" y2="63.5" width="0.1524" layer="91"/>
-<wire x1="76.2" y1="43.18" x2="81.28" y2="43.18" width="0.1524" layer="91"/>
-<wire x1="81.28" y1="43.18" x2="91.44" y2="43.18" width="0.1524" layer="91"/>
-<wire x1="91.44" y1="43.18" x2="91.44" y2="68.58" width="0.1524" layer="91"/>
-<wire x1="50.8" y1="63.5" x2="81.28" y2="63.5" width="0.1524" layer="91"/>
-<wire x1="81.28" y1="63.5" x2="81.28" y2="43.18" width="0.1524" layer="91"/>
-<junction x="81.28" y="43.18"/>
-<wire x1="91.44" y1="68.58" x2="71.12" y2="68.58" width="0.1524" layer="91"/>
-<wire x1="71.12" y1="68.58" x2="68.58" y2="68.58" width="0.1524" layer="91"/>
-<wire x1="91.44" y1="43.18" x2="99.06" y2="43.18" width="0.1524" layer="91"/>
-<junction x="91.44" y="43.18"/>
-<pinref part="U2" gate="G1" pin="-IN"/>
-<pinref part="U2" gate="G1" pin="OUT"/>
-<pinref part="R3" gate="G$1" pin="1"/>
-<junction x="71.12" y="68.58"/>
-<pinref part="R11" gate="G$1" pin="2"/>
-</segment>
-</net>
-<net name="N$3" class="0">
-<segment>
-<wire x1="50.8" y1="40.64" x2="60.96" y2="40.64" width="0.1524" layer="91"/>
-<wire x1="50.8" y1="40.64" x2="50.8" y2="38.1" width="0.1524" layer="91"/>
-<pinref part="U2" gate="G1" pin="+IN"/>
-<pinref part="C16" gate="G$1" pin="2"/>
-<wire x1="50.8" y1="38.1" x2="50.8" y2="33.02" width="0.1524" layer="91"/>
-<wire x1="43.18" y1="40.64" x2="50.8" y2="40.64" width="0.1524" layer="91"/>
-<junction x="50.8" y="40.64"/>
-<pinref part="R2" gate="G$1" pin="1"/>
-<junction x="50.8" y="38.1"/>
-</segment>
-</net>
-<net name="V+3" class="0">
-<segment>
-<wire x1="388.62" y1="106.68" x2="396.24" y2="106.68" width="0.1524" layer="91"/>
-<pinref part="C8" gate="G$1" pin="1"/>
-</segment>
-</net>
-<net name="V+4" class="0">
-<segment>
-<wire x1="388.62" y1="91.44" x2="396.24" y2="91.44" width="0.1524" layer="91"/>
-<pinref part="C13" gate="G$1" pin="1"/>
-</segment>
-</net>
+<junction x="388.62" y="91.44"/>
+<junction x="27.94" y="91.44"/>
+</segment>
+</net>
